Commit message: robot description

File: r1_description/robots/robot.urdf.xacro (robot description, xacro)
@@ -2,17 +2,9 @@
 <robot name="aion_r1" xmlns:xacro="http://wiki.ros.org/xacro">
   <!--  includes  -->
-  <xacro:include filename="$(find r1_description)/urdf/utils/utils.urdf.xacro"/>
   <xacro:include filename="$(find r1_description)/urdf/base/robot_base.urdf.xacro"/>
-  <xacro:include filename="$(find r1_description)/urdf/wheels/rover_wheel.urdf.xacro"/>
   <!--  argumentos  -->
   <xacro:arg name="robot_ns" default=""/>
   <xacro:arg name="prefix" default=""/>
-  <!--  Robot Parts  -->
-  <!--  Utils  -->
-  <xacro:utils/>
   <!--  Base  -->
   <xacro:robot_base/>
-  <!--  Wheels  -->
-  <xacro:rover_wheel parent="base_link2">
-  </xacro:rover_wheel>
 </robot>

File: r1_description/urdf/base/robot_base.urdf.xacro (robot description, xacro)
@@ -2,105 +2,9 @@
 <robot name="aion_r1" xmlns:xacro="http://wiki.ros.org/xacro">
   <xacro:macro name="robot_base">
-    <joint name="base_cover_link_joint" type="fixed">
-      <origin rpy="0.00000 0.00000 0.00000" xyz="0.00000 0.00000 0.05950"/>
-      <parent link="base_link2"/>
-      <child link="base_cover_link"/>
-    </joint>
-    <joint name="base_link2_joint" type="fixed">
-      <origin rpy="0.00000 0.00000 0.00000" xyz="0.00000 0.00000 0.11750"/>
-      <parent link="base_footprint"/>
-      <child link="base_link2"/>
-    </joint>
-    <joint name="batery_link_joint" type="fixed">
-      <origin rpy="0.00000 0.00000 0.00000" xyz="-0.08750 0.00000 0.08150"/>
-      <parent link="base_link2"/>
-      <child link="batery_link"/>
-    </joint>
-    <joint name="gps_link_joint" type="fixed">
-      <origin rpy="0.00000 0.00000 0.00000" xyz="0.03500 0.00000 0.09150"/>
-      <parent link="base_link2"/>
-      <child link="gps_link"/>
-    </joint>
-    <joint name="lidar_link_joint" type="fixed">
-      <origin rpy="0.00000 0.00000 0.00000" xyz="0.13000 0.00000 0.07750"/>
-      <parent link="base_link2"/>
-      <child link="lidar_link"/>
-    </joint>
-    <link name="base_footprint"/>
-    <link name="base_cover_link">
-      <collision name="base_cover_collision">
-        <origin rpy="0.00000 0.00000 0.00000" xyz="0.00000 0.00000 -0.00000"/>
+    <link name="robot_meshes">
+      <visual name="robot_link">
+        <origin rpy="0.000000 0.000000 0.000000" xyz="0.000000 0.000000 0.000000"/>
         <geometry>
-          <box size="0.41000 0.33000 0.00400"/>
-        </geometry>
-      </collision>
-      <inertial>
-        <inertia ixx="0.00227" ixy="0.00000" ixz="0.00000" iyy="0.00350" iyz="0.00000" izz="0.00577"/>
-        <origin rpy="0.00000 0.00000 0.00000" xyz="0.00000 0.00000 -0.00000"/>
-        <mass value="0.25000"/>
-      </inertial>
-      <visual name="base_cover">
-        <origin rpy="0.00000 0.00000 0.00000" xyz="0.00000 0.00000 -0.00000"/>
-        <material name="Material_white"/>
-        <geometry>
-          <box size="0.41000 0.33000 0.00400"/>
-        </geometry>
-      </visual>
-    </link>
-    <link name="base_link2">
-      <collision name="base_collision">
-        <origin rpy="0.00000 0.00000 0.00000" xyz="0.00000 0.00000 -0.00000"/>
-        <geometry>
-          <box size="0.40000 0.21000 0.11500"/>
-        </geometry>
-      </collision>
-      <inertial>
-        <inertia ixx="0.00955" ixy="0.00000" ixz="0.00000" iyy="0.02887" iyz="0.00000" izz="0.03402"/>
-        <origin rpy="0.00000 0.00000 0.00000" xyz="0.00000 0.00000 0.00000"/>
-        <mass value="2.00000"/>
-      </inertial>
-      <visual name="base">
-        <origin rpy="0.00000 0.00000 0.00000" xyz="0.00000 0.00000 0.00000"/>
-        <material name="Material_grey"/>
-        <geometry>
-          <box size="0.40000 0.21000 0.11500"/>
-        </geometry>
-      </visual>
-    </link>
-    <link name="batery_link">
-      <collision name="batery_collision">
-        <origin rpy="0.00000 0.00000 0.00000" xyz="-0.00000 0.00000 0.00000"/>
-        <geometry>
-          <box size="0.14500 0.05500 0.04000"/>
-        </geometry>
-      </collision>
-      <inertial>
-        <inertia ixx="0.00012" ixy="0.00000" ixz="0.00000" iyy="0.00057" iyz="0.00000" izz="0.00060"/>
-        <origin rpy="0.00000 0.00000 0.00000" xyz="0.00000 0.00000 0.00000"/>
-        <mass value="0.30000"/>
-      </inertial>
-      <visual name="batery">
-        <origin rpy="0.00000 0.00000 0.00000" xyz="-0.00000 0.00000 0.00000"/>
-        <material name="Material_black"/>
-        <geometry>
-          <box size="0.14500 0.05500 0.04000"/>
-        </geometry>
-      </visual>
-    </link>
-    <link name="gps_link">
-      <visual name="gps">
-        <origin rpy="0.00000 0.00000 0.00000" xyz="0.00000 0.00000 -0.00000"/>
-        <material name="Material_black"/>
-        <geometry>
-          <cylinder radius="0.05000" length="0.06000"/>
-        </geometry>
-      </visual>
-    </link>
-    <link name="lidar_link">
-      <visual name="lidar">
-        <origin rpy="0.00000 0.00000 0.00000" xyz="0.00000 0.00000 -0.00000"/>
-        <material name="Material_black"/>
-        <geometry>
-          <cylinder radius="0.02500" length="0.04000"/>
+          <mesh filename="file://$(find r1_description)/meshes/dae/chassis_link.dae" scale="1.000000 1.000000 1.000000"/>
         </geometry>
       </visual>
